File: Hardware/Kicad Files/MrKoh.kicad_sch (KiCad schematic)
At the start: 47 parts, among them J1 USB_C_Receptacle_USB2.0, J2 header, Q1 MMBT3904, SW1 RESET, SW2 BOOT, U1 USBLC6-2SC6, U2 ESP32-C3-FH4, U3 AZ1117-3.3, Y1 32K (C32346), Y2 40Mhz (C252256)

Commit message: Part issue
There was a problem with sourcing the original RGB part and changes to schematic, pcb, and fabrication files.  Production proofs were added.
Parts:
- D2: footprint LED_SMD:LED_WS2812B-2020_PLCC4_2.0x2.0mm -> LED_SMD:LED_WS2812B_PLCC4_5.0x5.0mm_P3.2mm
Changed lines of the file:
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@@
     (property "Reference" "D2" (id 0) (at 186.055 140.335 90))
     (property "Value" "WS2812B" (id 1) (at 184.785 130.175 0))
-    (property "Footprint" "LED_SMD:LED_WS2812B-2020_PLCC4_2.0x2.0mm" (id 2) (at 180.975 144.145 0)
+    (property "Footprint" "LED_SMD:LED_WS2812B_PLCC4_5.0x5.0mm_P3.2mm" (id 2) (at 180.975 144.145 0)
       (effects (font (size 1.27 1.27)) (justify left top) hide)
     )
@@
     )
     (path "/ebcc2821-4502-4f55-ac9c-2ba6e29aacd8"
-      (reference "D2") (unit 1) (value "WS2812B") (footprint "LED_SMD:LED_WS2812B-2020_PLCC4_2.0x2.0mm")
+      (reference "D2") (unit 1) (value "WS2812B") (footprint "LED_SMD:LED_WS2812B_PLCC4_5.0x5.0mm_P3.2mm")
     )
     (path "/6586ce7c-7ee1-4b58-b2ce-66c3da8cb1c8"
